File: HW/co_hw/7segments.kicad_sch (KiCad schematic)
At the start: 8 parts, among them U2 74HC595, U3 74HC595, U4 74HC595, U5 74HC595

Commit message: HW update.
Parts:
- added C16, C17, C18, C19: 100nF, symbol Device:C
Connections:
- net SR_RST: now reaches U4.10 (~{SRCLR})
- net SR_RST: now also U2.10 (~{SRCLR}), U3.10 (~{SRCLR}), U5.10 (~{SRCLR})
- net SR_CLK: now reaches U4.11 (SRCLK)
- net SR_CLK: now also U2.11 (SRCLK), U3.11 (SRCLK), U5.11 (SRCLK)
- net SR_LATCH: now reaches U4.12 (RCLK)
- net SR_LATCH: now also U2.12 (RCLK), U3.12 (RCLK), U5.12 (RCLK)
- net GND: now reaches U4.13 (~{OE})
- net GND: now also U2.13 (~{OE}), U2.8 (GND), U3.13 (~{OE}), U3.8 (GND), U4.8 (GND), U5.13 (~{OE}), U5.8 (GND), C16.2, C17.2, C18.2, C19.2
- net SR_2OUT: now reaches U4.14 (SER)
- net SR_2OUT: now also U3.9 (QH')
- net +3V3: now reaches U4.16 (VCC)
- net +3V3: now also U2.16 (VCC), U3.16 (VCC), U5.16 (VCC), C16.1, C17.1, C18.1, C19.1
- net SR_3OUT: now reaches U4.9 (QH')
- net SR_3OUT: now also U5.14 (SER)
- net SR_1OUT: now reaches U3.14 (SER)
- net SR_1OUT: now also U2.9 (QH')
- net SR_DATA_IN: now reaches U2.14 (SER)
- no-connect marks 0 -> 1
Other:
- note added: "SR_IN - DATA SR_CLK - CLOCK SR_RCLK - LATCH NORMAL HI/ WRITING LO SR_CLR - CLEAR HIGH RUNTIME / CLEAR LOW"
- moved on the sheet: AFF1, AFF2, D1, D2, U2, U3, U4, U5

Commit message: HW update.
Parts:
- removed D1: ~, Own_Library:KYX-1514YG, symbol Own_Library:KYX-1514YG
- added D5: ~, Own_Library:KYX-1514YG, symbol Own_Library:KYX-1514YG
- added R11, R12, R13, R14, R15, R16, R17, R18, R19, R20, R21, R22, R23, R24, R25, R26, R27, R28, R29, R30, R31, R32, R33, R34, R36, R37, R38, R39, R40, R41, R42, R43: 200, symbol Device:R
Connections:
- net QE_1R: now reaches AFF1.1 (e)
- net QE_1R: now also R15.2
- net QG_1R: now reaches AFF1.10 (g)
- net QG_1R: now also R13.2
- net QD_1R: now reaches AFF1.2 (d)
- net QD_1R: now also R16.2
- net QC_1R: now reaches AFF1.4 (c)
- net QC_1R: now also R11.2
- net QH_1R: now reaches AFF1.5 (DP)
- net QH_1R: now also R12.2
- net QB_1R: now reaches AFF1.6 (b)
- net QB_1R: now also R17.2
- net QA_1R: now reaches AFF1.7 (a)
- net QA_1R: now also R18.2
- net QF_1R: now reaches AFF1.9 (f)
- net QF_1R: now also R14.2
- net QE_2R: now reaches AFF2.1 (e)
- net QE_2R: now also R22.2
- net QG_2R: now reaches AFF2.10 (g)
- net QG_2R: now also R20.2
- net QD_2R: now reaches AFF2.2 (d)
- net QD_2R: now also R23.2
- net QC_2R: now reaches AFF2.4 (c)
- net QC_2R: now also R24.2
- net QH_2R: now reaches AFF2.5 (DP)
- net QH_2R: now also R19.2
- net QB_2R: now reaches AFF2.6 (b)
- net QB_2R: now also R25.2
- net QA_2R: now reaches AFF2.7 (a)
- net QA_2R: now also R26.2
- net QF_2R: now reaches AFF2.9 (f)
- net QF_2R: now also R21.2
- net QB_3: now reaches U4.1 (QB)
- net QB_3: now also R33.1
- net QA_3: now reaches U4.15 (QA)
- net QA_3: now also R34.1
- net QC_3: now reaches U4.2 (QC)
- net QC_3: now also R32.1
- net QD_3: now reaches U4.3 (QD)
- net QD_3: now also R31.1
- net QE_3: now reaches U4.4 (QE)
- net QE_3: now also R30.1
- net QF_3: now reaches U4.5 (QF)
- net QF_3: now also R29.1
- net QG_3: now reaches U4.6 (QG)
- net QG_3: now also R28.1
- net QH_3: now reaches U4.7 (QH)
- net QH_3: now also R27.1
- net QB_2: now reaches U3.1 (QB)
- net QB_2: now also R25.1
- net QA_2: now reaches U3.15 (QA)
- net QA_2: now also R26.1
- net QC_2: now reaches U3.2 (QC)
- net QC_2: now also R24.1
- net QD_2: now reaches U3.3 (QD)
- net QD_2: now also R23.1
- net QE_2: now reaches U3.4 (QE)
- net QE_2: now also R22.1
- net QF_2: now reaches U3.5 (QF)
- net QF_2: now also R21.1
- net QG_2: now reaches U3.6 (QG)
- net QG_2: now also R20.1
- net QH_2: now reaches U3.7 (QH)
- net QH_2: now also R19.1
- net QB_1: now reaches U2.1 (QB)
- net QB_1: now also R17.1
- net QA_1: now reaches U2.15 (QA)
- net QA_1: now also R18.1
- net QC_1: now reaches U2.2 (QC)
- net QC_1: now also R11.1
- net QD_1: now reaches U2.3 (QD)
- net QD_1: now also R16.1
- net QE_1: now reaches U2.4 (QE)
- net QE_1: now also R15.1
- net QF_1: now reaches U2.5 (QF)
- net QF_1: now also R14.1
- net QG_1: now reaches U2.6 (QG)
- net QG_1: now also R13.1
- net QH_1: now reaches U2.7 (QH)
- net QH_1: now also R12.1
- net QB_4: now reaches U5.1 (QB)
- net QB_4: now also R42.1
- net QA_4: now reaches U5.15 (QA)
- net QA_4: now also R43.1
- net QC_4: now reaches U5.2 (QC)
- net QC_4: now also R41.1
- net QD_4: now reaches U5.3 (QD)
- net QD_4: now also R40.1
- net QE_4: now reaches U5.4 (QE)
- net QE_4: now also R39.1
- net QF_4: now reaches U5.5 (QF)
- net QF_4: now also R38.1
- net QG_4: now reaches U5.6 (QG)
- net QG_4: now also R37.1
- net QH_4: now reaches U5.7 (QH)
- net QH_4: now also R36.1
- net SR_CLK renamed G_SR_CLK
- net SR_DATA_IN renamed G_SR_DATA_IN
- net SR_LATCH renamed G_SR_LATCH
- net SR_RST renamed G_SR_RST
- new net QA_3R: D5.1 (A), R34.2
- new net QA_4R: D5.9 (I), R43.2
- new net QB_3R: D5.2 (B), R33.2
- new net QB_4R: D5.10 (K), R42.2
- new net QC_3R: D5.3 (C), R32.2
- new net QC_4R: R41.2
- new net QD_3R: D5.4 (D), R31.2
- new net QD_4R: R40.2
- new net QE_3R: D5.5 (E), R30.2
- new net QE_4R: R39.2
- new net QF_3R: D5.6 (F), R29.2
- new net QF_4R: R38.2
- new net QG_3R: D5.7 (G), R28.2
- new net QG_4R: R37.2
- new net QH_3R: D5.8 (H), R27.2
- new net QH_4R: R36.2
- no-connect marks 1 -> 7
Other:
- moved on the sheet: D2, U2, U3, U4, U5

Commit message: HW update.
Connections:
- net GND: now also AFF1.3 (C.K.), AFF1.8 (C.K.), AFF2.3 (C.K.), AFF2.8 (C.K.), D5.11 (GND), D5.12 (GND)
Other:
- moved on the sheet: AFF1, AFF2, D5
