File: HW/co_hw/co_hw.kicad_sch (KiCad schematic)
At the start: 6 parts, among them SW1 RotaryEncoder_Switch, U1 STM32F103C8Tx, U2 74HC595, U3 74HC595, U4 74HC595, U5 74HC595

Commit message: HW init.
Parts:
- removed SW1: RotaryEncoder_Switch, symbol Device:RotaryEncoder_Switch
- removed U1: STM32F103C8Tx, Package_QFP:LQFP-48_7x7mm_P0.5mm, symbol MCU_ST_STM32F1:STM32F103C8Tx
- removed U2, U3, U4, U5: 74HC595, symbol 74xx:74HC595
Other:
- added sheet microcontroler (untitled.kicad_sch)
- added sheet power_supply (power_supply_sch.kicad_sch)

Commit message: Update HW
Other:
- added sheet 7segments (7segments.kicad_sch)
- sheet microcontroler: file untitled.kicad_sch -> microcontroler.kicad_sch
Changed lines of the file:
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@@
 			)
 		)
-		(property "Sheetfile" "untitled.kicad_sch"
+		(property "Sheetfile" "microcontroler.kicad_sch"
 			(at 107.95 85.6746 0)
 			(effects
@@
 			(effects
 				(font
+					(size 1.27 1.27)
+				)
+				(justify left top)
+			)
+		)
+		(instances
+			(project "co_hw"
+				(path "/ccf087ed-af29-4b01-8b29-73c7633787ca"
+					(page "4")
+				)
+			)
+		)
+	)
+	(sheet
+		(at 163.83 52.07)
+		(size 40.64 38.1)
+		(exclude_from_sim no)
+		(in_bom yes)
+		(on_board yes)
+		(dnp no)
+		(fields_autoplaced yes)
+		(stroke
+			(width 0.1524)
+			(type solid)
+		)
+		(fill
+			(color 0 0 0 0.0000)
+		)
+		(property "Sheetname" "7segments"
+			(at 163.83 51.3584 0)
+			(effects
+				(font
+					(size 1.27 1.27)
+				)
+				(justify left bottom)
+			)
+		)
+		(property "Sheetfile" "7segments.kicad_sch"
+			(at 163.83 90.7546 0)
+			(effects
+				(font

Commit message: HW update.
Other:
- added sheet sensors (sensors.kicad_sch)
- sheet microcontroler ports: added H_ONE_WIRE, H_TIM3_PWM_BUZZER; removed none
Changed lines of the file:
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@@
 	(generator_version "9.0")
 	(paper "A4")
+	(wire
+		(pts
+			(xy 148.59 53.34) (xy 161.29 53.34)
+		)
+		(stroke
+			(width 0)
+			(type default)
+		)
+	)
+	(wire
+		(pts
+			(xy 148.59 55.88) (xy 161.29 55.88)
+		)
+		(stroke
+			(width 0)
+			(type default)
+		)
+	)
 	(sheet
 		(at 107.95 48.26)
@@
 			)
 		)
+		(pin "H_ONE_WIRE" bidirectional
+			(at 148.59 53.34 0)
+			(effects
+				(font
+					(size 1.27 1.27)
+				)
+				(justify right)
+			)
+		)
+		(pin "H_TIM3_PWM_BUZZER" output
+			(at 148.59 55.88 0)
+			(effects
+				(font
+					(size 1.27 1.27)
+				)
+				(justify right)
+			)
+		)
 		(instances
 			(project "co_hw"
@@
 	)
 	(sheet
-		(at 163.83 52.07)
-		(size 40.64 38.1)
+		(at 161.29 73.66)
+		(size 34.29 20.32)
 		(exclude_from_sim no)
 		(in_bom yes)
@@
 		)
 		(property "Sheetname" "7segments"
-			(at 163.83 51.3584 0)
+			(at 161.29 72.9484 0)
 			(effects
 				(font
@@
 		)
 		(property "Sheetfile" "7segments.kicad_sch"
-			(at 163.83 90.7546 0)
+			(at 161.29 94.5646 0)
 			(effects
 				(font
@@
 				)
 			)
+		)
+	)
+	(sheet
+		(at 161.29 48.26)
+		(size 34.29 20.32)
+		(exclude_from_sim no)
+		(in_bom yes)
+		(on_board yes)
+		(dnp no)
+		(fields_autoplaced yes)
+		(stroke
+			(width 0.1524)
+			(type solid)
+		)
+		(fill
+			(color 0 0 0 0.0000)
+		)
+		(property "Sheetname" "sensors"
+			(at 161.29 47.5484 0)
+			(effects
+				(font
+					(size 1.27 1.27)
+				)
+				(justify left bottom)
+			)
+		)
+		(property "Sheetfile" "sensors.kicad_sch"
+			(at 161.29 69.1646 0)
+			(effects
+				(font
+					(size 1.27 1.27)
+				)
+				(justify left top)
+			)
+		)
+		(pin "H_ONE_WIRE" bidirectional
+			(at 161.29 53.34 180)
+			(effects
+				(font
+					(size 1.27 1.27)
+				)
+				(justify left)
+			)
+		)
+		(pin "H_TIM3_PWM_BUZZER" input
+			(at 161.29 55.88 180)
+			(effects
+				(font
+					(size 1.27 1.27)
+				)
+				(justify left)
+			)
+		)
+		(instances
+			(project "co_hw"
+				(path "/ccf087ed-af29-4b01-8b29-73c7633787ca"
+					(page "5")
+				)
+			)

Commit message: HW update
Other:
- sheet microcontroler ports: added I2C2{SDA SCL}, TIM4_PWM_LED{_R _G _B}; removed none
- sheet sensors ports: added I2C2{SDA SCL}; removed none
Changed lines of the file:
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@@
+	(wire
+		(pts
+			(xy 148.59 58.42) (xy 161.29 58.42)
+		)
+		(stroke
+			(width 0)
+			(type default)
+		)
+	)
 	(wire
 		(pts
@@
 		(pin "H_TIM3_PWM_BUZZER" output
 			(at 148.59 55.88 0)
+			(effects
+				(font
+					(size 1.27 1.27)
+				)
+				(justify right)
+			)
+		)
+		(pin "I2C2{SDA SCL}" bidirectional
+			(at 148.59 58.42 0)
+			(effects
+				(font
+					(size 1.27 1.27)
+				)
+				(justify right)
+			)
+		)
+		(pin "TIM4_PWM_LED{_R _G _B}" output
+			(at 148.59 60.96 0)
 			(effects
 				(font
@@
 			(effects
 				(font
+					(size 1.27 1.27)
+				)
+				(justify left)
+			)
+		)
+		(pin "I2C2{SDA SCL}" bidirectional
+			(at 161.29 58.42 180)
+			(effects
+				(font
