File: HW/co_hw/microcontroler.kicad_sch (KiCad schematic)
At the start: 26 parts, among them J2 DS18B20, J3 DS18B20, J4 PRESSURE_SENSOR, J5 PWM, J7 Programmer, SW1 RotaryEncoder_Switch, SW2 SW_DIP_x03, SW3 SW_Push, U1 STM32F103C8Tx, U6 W25Q32JVSS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

Commit message: HW update.
Parts:
- added C12, C13, C14, C15: 100nF, symbol Device:C
- added R10, R7, R8, R9: 10k, symbol Device:R
- added R5, R6: 100, symbol Device:R
Connections:
- net +3V3: now also SW1.S2, U6.8 (VCC), C12.1, R10.2, R7.1, R8.2
- net GND: now also SW1.C, U6.4 (GND), C12.2, C13.2, C14.2, C15.2, R9.1
- net TIM2_ENCODER_CH1: now also C13.1, R5.2, R7.2
- net TIM2_ENCODER_CH2: now also C14.1, R6.2, R8.1
- net W25Q32_CS: now reaches U6.1 (~{CS})
- net W25Q32_MISO: now reaches U6.2 (DO/IO_{1})
- net /WP: now reaches U6.3 (~{WP}/IO_{2})
- net /WP: now also R10.1
- net W25Q32_MOSI: now reaches U6.5 (DI/IO_{0})
- net W25Q32_CLK: now reaches U6.6 (CLK)
- net W25Q32_RST: now reaches U6.7 (~{HOLD}/~{RESET}/IO_{3})
- net at SW1.A: now also R5.1
- net at SW1.B: now also R6.1
- net SW1: now reaches SW1.S1
- net SW1: now also C15.1, R9.2
Other:
- moved on the sheet: BZ1, SW1, U6

Commit message: HW update.
Parts:
- removed BZ1: ~, Own_Library:SFM-27-W, symbol Own_Library:SFM-27
- removed J2: DS18B20, Connector_Molex:Molex_Mini-Fit_Sr_42820-32XX_1x03_P10.00mm_Horizontal_ThermalVias, symbol Connector:Conn_01x03_Socket
- removed J3: DS18B20, symbol Connector:Conn_01x03_Socket
- removed J4: PRESSURE_SENSOR, symbol Connector:Conn_01x03_Socket
- removed J5: PWM, symbol Connector:Conn_01x03_Socket
Connections:
- net 3V3 is gone; now on net +3V3: J7.7 (Pin_7)
- net SPI2_MISO: now also U1.27 (PB14); no longer U1.37 (PA14)
- net SPI2_MOSI: now also U1.28 (PB15); no longer U1.38 (PA15)
- net SPI2_SCK: now also U1.26 (PB13); no longer U1.34 (PA13)
- net SWCLK: now also U1.37 (PA14); no longer U1.27 (PB14)
- net SWDIO: now also U1.34 (PA13); no longer U1.26 (PB13)
- net TIM2_ENCODER_CH1: now also U1.38 (PA15)
- net TIM2_ENCODER_CH2: now also U1.39 (PB3)
- net U_RX: now also U1.30 (PA9)
- net U_TX: now also U1.31 (PA10)
- net W25Q32_CS: now also U1.18 (PB0)
- net W25Q32_RST: now also U1.4 (PC15)
- net G_PRESSURE_SENSOR_ANALOG: now reaches U1.10 (PA0)
- net G_SERVO_MOTOR_PWM: now reaches U1.13 (PA3)
- net CC1101_CS: now reaches U1.19 (PB1)
- net G_SR_LATCH: now reaches U1.2 (PC13)
- net CC1101_GD00: now reaches U1.20 (PB2)
- net G_SR_RST: now reaches U1.3 (PC14)
- net 5V renamed VCC_5V
- net ONE_WIRE renamed H_ONE_WIRE
- net PWM_BUZZER renamed CC1101_GD02
- net PWM_LED_B renamed TIM4_PWM_LED_B
- net PWM_LED_G renamed TIM4_PWM_LED_G
- net PWM_LED_R renamed TIM4_PWM_LED_R
- net SPI1_MISO renamed H_TIM3_PWM_BUZZER
- net SPI1_MOSI renamed G_SR_DATA_IN
- net SPI1_SCK renamed G_SR_CLK
- net VCCA renamed VCCA_3V3
Other:
- moved on the sheet: R2, R3, R4

Commit message: HW update.
Connections:
- net I2C2_SCL is gone; now on net I2C1_SCL: U1.21 (PB10)
- net I2C2_SDA is gone; now on net I2C1_SDA: U1.22 (PB11)
- net GND: now also U1.23 (VSS), U1.35 (VSS), U1.47 (VSS)
Changed lines of the file:
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@@
 	(wire
 		(pts
-			(xy 148.59 130.81) (xy 148.59 132.08)
+			(xy 148.59 130.81) (xy 148.59 134.62)
 		)
 		(stroke
@@
 		(pts
 			(xy 119.38 21.59) (xy 121.92 21.59)
+		)
+		(stroke
+			(width 0)
+			(type default)
+		)
+	)
+	(wire
+		(pts
+			(xy 144.78 134.62) (xy 148.59 134.62)
 		)
 		(stroke
@@
 		)
 	)
+	(label "I2C2_SDA"
+		(at 60.96 107.95 180)
+		(effects
+			(font
+				(size 1.27 1.27)
+			)
+			(justify right bottom)
+		)
+	)
 	(label "SW1"
 		(at 227.33 66.04 0)
@@
 			)
 			(justify left bottom)
+		)
+	)
+	(label "I2C2_SCL"
+		(at 60.96 105.41 180)
+		(effects
+			(font
+				(size 1.27 1.27)
+			)
+			(justify right bottom)
 		)
 	)
@@
 					(unit 1)
 				)
+			)
+		)
+	)
+	(symbol
+		(lib_id "power:GND")
+		(at 144.78 134.62 0)
+		(unit 1)
+		(exclude_from_sim no)
+		(in_bom yes)
+		(on_board yes)
+		(dnp no)
+		(fields_autoplaced yes)
+		(property "Reference" "#PWR048"
+			(at 144.78 140.97 0)
+			(effects
+				(font
+					(size 1.27 1.27)
+				)
+				(hide yes)
+			)
+		)
+		(property "Value" "GND"
+			(at 144.78 139.7 0)
+			(effects
+				(font
+					(size 1.27 1.27)
+				)
+			)
+		)
+		(property "Footprint" ""
+			(at 144.78 134.62 0)
+			(effects
+				(font
+					(size 1.27 1.27)
+				)
+				(hide yes)
+			)
+		)
+		(property "Datasheet" ""
+			(at 144.78 134.62 0)
+			(effects
+				(font
+					(size 1.27 1.27)
+				)
+				(hide yes)
+			)
+		)
+		(property "Description" "Power symbol creates a global label with name \"GND\" , ground"
+			(at 144.78 134.62 0)
+			(effects
+				(font
+					(size 1.27 1.27)
+				)
+				(hide yes)
+			)
+		)
+		(pin "1"
+		)
+		(instances
+			(project "co_hw"
+				(path "/ccf087ed-af29-4b01-8b29-73c7633787ca/03ef4d79-8cc0-4095-8497-12b728c23f87"
+					(reference "#PWR048")
+					(unit 1)
+				)

Commit message: HW update
Connections:
- net I2C1_SCL renamed I2C2.SCL
- net I2C1_SDA renamed I2C2.SDA
- net U_RX renamed UART_RX
- net U_TX renamed UART_TX
Other:
- moved on the sheet: R3, R4

Commit message: Update HW.
Parts:
- added R44: 0R, symbol Device:R
- added U10: ~, symbol Own_Library:CC1101_Module
Connections:
- net W25Q32_CLK is gone; now on net CC1101_SCK: U6.6 (CLK)
- net W25Q32_MISO is gone; now on net CC1101_MISO: U6.2 (DO/IO_{1})
- net W25Q32_MOSI is gone; now on net CC1101_MOSI: U6.5 (DI/IO_{0})
- net +3V3: now also U10.2 (VCC)
- net CC1101_CS: now also U10.8 (CSN)
- net CC1101_GD00: now also U10.7 (GDO0)
- net CC1101_GD02: now also U10.6 (GDO2)
- net GND: now also U10.1 (GND)
- net nRST: now also R44.1
- net at C3.1, SW3.2, U1.7 (NRST): now also R44.2
- net SPI2_MISO renamed CC1101_MISO
- net CC1101_MISO: now also U10.5 (SO)
- net SPI2_MOSI renamed CC1101_MOSI
- net CC1101_MOSI: now also U10.3 (SI)
- net SPI2_SCK renamed CC1101_SCK
- net CC1101_SCK: now also U10.4 (SCLK)

Commit message: Update HW
Connections:
- net RELAY_2: now reaches U1.25 (PB12)
- net RELAY_1: now reaches U1.46 (PB9)
Other:
- note added: "max 25mA"
- note added: "max 35mA"
Changed lines of the file:
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@@
 	(generator_version "9.0")
 	(paper "A4")
+	(text "max 25mA"
+		(exclude_from_sim no)
+		(at 265.684 20.066 0)
+		(effects
+			(font
+				(size 1.27 1.27)
+			)
+		)
+	)
+	(text "max 35mA"
+		(exclude_from_sim no)
+		(at 263.652 128.778 0)
+		(effects
+			(font
+				(size 1.27 1.27)
+			)
+		)
+	)
 	(junction
 		(at 254 99.06)
@@
 	(wire
 		(pts
+			(xy 115.57 115.57) (xy 130.81 115.57)
+		)
+		(stroke
+			(width 0)
+			(type default)
+		)
+	)
+	(wire
+		(pts
 			(xy 119.38 34.29) (xy 119.38 31.75)
 		)
@@
 		(pts
 			(xy 146.05 44.45) (xy 148.59 44.45)
+		)
+		(stroke
+			(width 0)
+			(type default)
+		)
+	)
+	(wire
+		(pts
+			(xy 115.57 107.95) (xy 130.81 107.95)
 		)
 		(stroke
@@
 		)
 	)
+	(global_label "RELAY_2"
+		(shape output)
+		(at 115.57 115.57 180)
+		(fields_autoplaced yes)
+		(effects
+			(font
+				(size 1.27 1.27)
+			)
+			(justify right)
+		)
+		(property "Intersheetrefs" "${INTERSHEET_REFS}"
+			(at 104.7834 115.57 0)
+			(effects
+				(font
+					(size 1.27 1.27)
+				)
+				(justify right)
+				(hide yes)
+			)
+		)
+	)
 	(global_label "G_PRESSURE_SENSOR_ANALOG"
 		(shape input)
@@
 				(hide yes)
 			)
+		)
+	)
+	(global_label "RELAY_1"
+		(shape output)
+		(at 115.57 107.95 180)
+		(fields_autoplaced yes)
+		(effects
+			(font
+				(size 1.27 1.27)
+			)
+			(justify right)
+		)
+		(property "Intersheetrefs" "${INTERSHEET_REFS}"
+			(at 104.7834 107.95 0)
+			(effects
+				(font
+					(size 1.27 1.27)
+				)
+				(justify right)
+				(hide yes)
+			)
