File: HW/co_hw/power_supply_sch.kicad_sch (KiCad schematic)
At the start: 9 parts, among them J1 Screw_Terminal_OUTPUT, J6 Screw_Terminal_INPUT, K1 SANYOU_SRD_Form_C

Commit message: HW update.
Parts:
- added D3: 1N4001, Diode_THT:D_DO-41_SOD81_P10.16mm_Horizontal, symbol Diode:1N4001
Changed lines of the file:
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@@
+	)
+	(symbol
+		(lib_id "Diode:1N4001")
+		(at 69.85 88.9 0)
+		(unit 1)
+		(exclude_from_sim no)
+		(in_bom yes)
+		(on_board yes)
+		(dnp no)
+		(fields_autoplaced yes)
+		(property "Reference" "D3"
+			(at 69.85 82.55 0)
+			(effects
+				(font
+					(size 1.27 1.27)
+				)
+			)
+		)
+		(property "Value" "1N4001"
+			(at 69.85 85.09 0)
+			(effects
+				(font
+					(size 1.27 1.27)
+				)
+			)
+		)
+		(property "Footprint" "Diode_THT:D_DO-41_SOD81_P10.16mm_Horizontal"
+			(at 69.85 88.9 0)
+			(effects
+				(font
+					(size 1.27 1.27)
+				)
+				(hide yes)
+			)
+		)
+		(property "Datasheet" "http://www.vishay.com/docs/88503/1n4001.pdf"
+			(at 69.85 88.9 0)
+			(effects
+				(font
+					(size 1.27 1.27)
+				)
+				(hide yes)
+			)
+		)
+		(property "Description" "50V 1A General Purpose Rectifier Diode, DO-41"
+			(at 69.85 88.9 0)
+			(effects
+				(font
+					(size 1.27 1.27)
+				)
+				(hide yes)
+			)
+		)
+		(property "Sim.Device" "D"
+			(at 69.85 88.9 0)
+			(effects
+				(font
+					(size 1.27 1.27)
+				)
+				(hide yes)
+			)
+		)
+		(property "Sim.Pins" "1=K 2=A"
+			(at 69.85 88.9 0)
+			(effects
+				(font
+					(size 1.27 1.27)
+				)
+				(hide yes)
+			)
+		)
+		(pin "2"
+		)
+		(pin "1"
+		)
+		(instances
+			(project ""
+				(path "/ccf087ed-af29-4b01-8b29-73c7633787ca/08357ce8-a351-434e-a3f4-1502cd6508fc"
+					(reference "D3")
+					(unit 1)
+				)
+			)
+		)
 	)
 	(symbol

Commit message: HW update.
Parts:
- added D4: 1N4001, Diode_THT:D_DO-41_SOD81_P10.16mm_Horizontal, symbol Diode:1N4001
- added J8: Screw_Terminal_OUTPUT, symbol Connector:Screw_Terminal_01x03
- added K2: SANYOU_SRD_Form_C, Relay_THT:Relay_SPDT_SANYOU_SRD_Series_Form_C, symbol Relay:SANYOU_SRD_Form_C
Connections:
- net at C1.2, FL1.2, J1.2 (Pin_2)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: now also J8.2 (Pin_2)

Commit message: Update HW.
Connections:
- net at K2.3: now also J8.3 (Pin_3)
- net at J1.1 (Pin_1), J6.1 (Pin_1): now also J8.1 (Pin_1)
Changed lines of the file:
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@@
+	)
+	(junction
+		(at 41.91 62.23)
+		(diameter 0)
+		(color 0 0 0 0)
 	)
 	(junction
@@
 	(wire
 		(pts
+			(xy 41.91 62.23) (xy 41.91 120.65)
+		)
+		(stroke
+			(width 0)
+			(type default)
+		)
+	)
+	(wire
+		(pts
 			(xy 69.85 41.91) (xy 69.85 39.37)
 		)
@@
 	(wire
 		(pts
+			(xy 41.91 120.65) (xy 31.75 120.65)
+		)
+		(stroke
+			(width 0)
+			(type default)
+		)
+	)
+	(wire
+		(pts
 			(xy 148.59 34.29) (xy 151.13 34.29)
 		)
@@
 	(wire
 		(pts
+			(xy 57.15 115.57) (xy 57.15 104.14)
+		)
+		(stroke
+			(width 0)
+			(type default)
+		)
+	)
+	(wire
+		(pts
 			(xy 86.36 34.29) (xy 86.36 41.91)
 		)
@@
 		)
 		(stroke
+			(width 0)
+			(type default)
+		)
+	)
+	(wire
+		(pts
+			(xy 31.75 115.57) (xy 57.15 115.57)
+		)
+		(stroke

Commit message: Update HW
Parts:
- added U9: TPS5430DDA, Package_SO:TI_SO-PowerPAD-8_ThermalVias, symbol Regulator_Switching:TPS5430DDA
Connections:
- net GND: now also D3.2 (A), D4.2 (A), K1.2, K2.2
- net RELAY_2: now reaches K2.5
- net RELAY_2: now also D4.1 (K)
- net RELAY_1: now reaches K1.5
- net RELAY_1: now also D3.1 (K)
Other:
- note added: "120mA/3V"
- moved on the sheet: D3, D4
