File: HW/co_hw/sensors.kicad_sch (KiCad schematic)
At the start: 12 parts, among them J2 DS18B20, J3 DS18B20, J4 PRESSURE_SENSOR, J5 SERVO, Q1 2N7002, U7 BME280

Commit message: HW update.
Parts:
- added U8: SCD41, Own_Library:MODULE_SCD41, symbol Own_Library:SCD41
Changed lines of the file:
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@@
+	)
+	(symbol
+		(lib_id "Own_Library:SCD41")
+		(at 110.49 59.69 90)
+		(unit 1)
+		(exclude_from_sim no)
+		(in_bom yes)
+		(on_board yes)
+		(dnp no)
+		(fields_autoplaced yes)
+		(property "Reference" "U8"
+			(at 118.11 58.4199 90)
+			(effects
+				(font
+					(size 1.27 1.27)
+				)
+				(justify right)
+			)
+		)
+		(property "Value" "SCD41"
+			(at 118.11 60.9599 90)
+			(effects
+				(font
+					(size 1.27 1.27)
+				)
+				(justify right)
+			)
+		)
+		(property "Footprint" "Own_Library:MODULE_SCD41"
+			(at 110.49 59.69 0)
+			(effects
+				(font
+					(size 1.27 1.27)
+				)
+				(hide yes)
+			)
+		)
+		(property "Datasheet" "https://sensirion.com/media/documents/48C4B7FB/67FE0194/CD_DS_SCD4x_Datasheet_D1.pdf"
+			(at 110.49 59.69 0)
+			(effects
+				(font
+					(size 1.27 1.27)
+				)
+				(hide yes)
+			)
+		)
+		(property "Description" "Optical CO2 sensor"
+			(at 110.49 59.69 0)
+			(effects
+				(font
+					(size 1.27 1.27)
+				)
+				(hide yes)
+			)
+		)
+		(pin "1"
+		)
+		(pin "3"
+		)
+		(pin "2"
+		)
+		(pin "4"
+		)
+		(instances
+			(project ""
+				(path "/ccf087ed-af29-4b01-8b29-73c7633787ca/f3023918-9a15-4959-ba9c-d0d2bdfe9fec"
+					(reference "U8")
+					(unit 1)
+				)
+			)
+		)
 	)
 	(symbol

Commit message: HW update
Connections:
- net I2C2.SCL: now reaches U8.3 (SCL)
- net I2C2.SDA: now reaches U8.4 (SDA)
Changed lines of the file:
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@@
 		(color 0 0 0 0)
 	)
+	(bus_entry
+		(at 76.2 75.692)
+		(size 2.54 2.54)
+		(stroke
+			(width 0)
+			(type default)
+		)
+	)
+	(bus_entry
+		(at 76.2 76.708)
+		(size 2.54 2.54)
+		(stroke
+			(width 0)
+			(type default)
+		)
+	)
 	(wire
 		(pts
@@
 	(wire
 		(pts
+			(xy 78.74 78.74) (xy 111.76 78.74)
+		)
+		(stroke
+			(width 0)
+			(type default)
+		)
+	)
+	(wire
+		(pts
 			(xy 102.87 25.4) (xy 102.87 27.94)
 		)
@@
 		)
 	)
+	(bus
+		(pts
+			(xy 76.2 75.692) (xy 76.2 76.708)
+		)
+		(stroke
+			(width 0)
+			(type default)
+		)
+	)
 	(wire
 		(pts
@@
 	(wire
 		(pts
+			(xy 78.74 82.55) (xy 114.3 82.55)
+		)
+		(stroke
+			(width 0)
+			(type default)
+		)
+	)
+	(wire
+		(pts
+			(xy 78.74 78.232) (xy 78.74 78.74)
+		)
+		(stroke
+			(width 0)
+			(type default)
+		)
+	)
+	(wire
+		(pts
 			(xy 38.1 76.2) (xy 41.91 76.2)
 		)
@@
 		)
 	)
+	(bus
+		(pts
+			(xy 76.2 73.66) (xy 76.2 75.692)
+		)
+		(stroke
+			(width 0)
+			(type default)
+		)
+	)
 	(wire
 		(pts
@@
 	(wire
 		(pts
+			(xy 78.74 79.248) (xy 78.74 82.55)
+		)
+		(stroke
+			(width 0)
+			(type default)
+		)
+	)
+	(wire
+		(pts
 			(xy 242.57 115.57) (xy 242.57 118.11)
 		)
@@
 		)
 	)
+	(bus
+		(pts
+			(xy 76.2 76.708) (xy 76.2 81.28)
+		)
+		(stroke
+			(width 0)
+			(type default)
+		)
+	)
+	(wire
+		(pts
+			(xy 114.3 82.55) (xy 114.3 72.39)
+		)
+		(stroke
+			(width 0)
+			(type default)
+		)
+	)
 	(wire
 		(pts
@@
 		(pts
 			(xy 72.39 25.4) (xy 72.39 27.94)
+		)
+		(stroke
+			(width 0)
+			(type default)
+		)
+	)
+	(wire
+		(pts
+			(xy 111.76 72.39) (xy 111.76 78.74)
+		)
+		(stroke
+			(width 0)
+			(type default)
+		)
+	)
+	(bus
+		(pts
+			(xy 74.93 73.66) (xy 76.2 73.66)
 		)
 		(stroke
@@
 		)
 	)
+	(label "I2C2.SDA"
+		(at 96.52 82.55 0)
+		(effects
+			(font
+				(size 1.27 1.27)
+			)
+			(justify left bottom)
+		)
+	)
 	(label "SERVO_MOTOR_GND"
 		(at 228.6 59.69 0)
@@
 			)
 			(justify right bottom)
+		)
+	)
+	(label "I2C2.SCL"
+		(at 96.52 78.74 0)
+		(effects
+			(font
+				(size 1.27 1.27)
+			)
+			(justify left bottom)
 		)
 	)
@@
 		)
 	)
+	(hierarchical_label "I2C2{SDA SCL}"
+		(shape bidirectional)
+		(at 74.93 73.66 180)
+		(effects
+			(font
+				(size 1.27 1.27)
+			)
+			(justify right)
+		)
+	)

Commit message: Update HW
Other:
- note added: "max 20mA"
Changed lines of the file:
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@@
 	(generator_version "9.0")
 	(paper "A4")
+	(text "max 20mA"
+		(exclude_from_sim no)
+		(at 93.726 70.866 0)
+		(effects
+			(font
+				(size 1.27 1.27)
+			)
+		)
+	)
 	(junction
 		(at 102.87 27.94)
